Commit message: add Jacobian in ForwardKinematics.vue

File: public/industry/urdf/robot.urdf (robot description, URDF)
Before this commit: robot ER15-1400, 7 links, 6 joints
Joints:
- joint joint_6: origin xyz=0.1 0 0 rpy=-0.0013162 0 0 -> xyz=0.1 0 0 rpy=1.5708 0 1.5708

Commit message: remove something useless

File: public/industry/urdf/robot.urdf (robot description, URDF)
Before this commit: robot ER15-1400, 7 links, 6 joints
Links:
- link base_link: geometry collision mesh filename=package://meshes/base_link.STL; visual mesh filename=package://meshes/base_link.STL
- link link_1: geometry collision mesh filename=package://meshes/link_1.STL; visual mesh filename=package://meshes/link_1.STL
- link link_2: geometry collision mesh filename=package://meshes/link_2.STL; visual mesh filename=package://meshes/link_2.STL
- link link_3: geometry collision mesh filename=package://meshes/link_3.STL; visual mesh filename=package://meshes/link_3.STL
- link link_4: geometry collision mesh filename=package://meshes/link_4.STL; visual mesh filename=package://meshes/link_4.STL
- link link_5: geometry collision mesh filename=package://meshes/link_5.STL; visual mesh filename=package://meshes/link_5.STL
- link link_6: geometry collision mesh filename=package://meshes/link_6.STL; visual mesh filename=package://meshes/link_6.STL
